Commit message: env repaired

File: cartpole2.urdf (robot description, URDF)
Before this commit: robot physics, 4 links, 3 joints
Links:
- link cart: mass 1 -> 100
- link slideBar: mass 10000 -> 0; geometry visual box size=15 0.05 0.05

Commit message: Update a SQP model and MPPI model

File: cartpole2.urdf (robot description, URDF)
Before this commit: robot physics, 4 links, 3 joints
Links:
- link cart: mass 100 -> 1
- link pole: mass 10 -> 0.1
- link pole2: mass 10 -> 0.1
- link slideBar: geometry visual box size=30 0.05 0.05
